File: 477ProjectEagle/477ProjectSchematic.sch (EAGLE design)
At the start: 78 parts, among them J1 POWER_JACK_BAT, J2 POWER_JACK_12VOUT, J3 RJ11-6PTH, Q1 AO4419, X1 22-23-2051, X10 MOTORS

Commit message: Fixed some main PCB things
Put standoff holes in board. Fixed encoder headers so that there are 4
banks of 3 holed headers. (2 three holed headers per encoder.)
Parts:
- removed ENCODER: 22-23-2021, con-molex:22-23-2021
- added JP1, JP2, JP3, JP4: (no value), pinhead:PINHD-1X3
Connections:
- removed net N$72: SV8.6, U$1.IC2/*U1CTS/INT2/RD9
- new net N$12: JP3.1, SV8.6, U$1.IC2/*U1CTS/INT2/RD9
- net +5V: now also JP1.2, JP2.2, JP3.2, JP4.2
- net GND: now also JP1.3, JP2.3, JP3.3, JP4.3
- net N$70: now also JP2.1; no longer ENCODER-1.S
- net N$71: now also JP1.1; no longer ENCODER-2.S
- net N$73: now also JP4.1
