File: 477ProjectEagle/477ProjectSchematic.sch (EAGLE design)
At the start: 81 parts, among them J1 POWER_JACK_BAT, J2 POWER_JACK_12VOUT, J3 RJ11-6PTH, Q1 AO4419, X1 22-23-2051, X10 MOTORS

Commit message: Did some verification of the schematic
Fixed resistor values for power supplies. Fixed the max 233 chip
connections and the DB9 connections. Verified everything on the main PCB
schematic except reset button and programming header.
Parts:
- added J4: POWER_JACK_BAT, SparkFun-Connectors:POWER_JACKPTH
- added U$5: 0.1uF, MinotaurParts:C-US-1206
- CVCC12: value 740nF -> 470nF
- R1_5: value (none) -> 105k
- R2_5: value (none) -> 20k
- U$45, U$46, U$47, U$48, U$49: value 10uF -> 0.1uF
Connections:
- removed net N$86: J3.3
- new net N$13: U$39.V-, U$39.V-2
- new net N$62: U$39.C2-, U$39.CS-
- new net N$72: U$39.C2+, U$39.C2+2
- net +3V3: now also J4.PWR
- net +7V: now also U$5.1
- net GND: now also J3.3, J4.GND, J4.GNDBREAK, U$5.2, X4.5; no longer X4.1

Commit message: PCB is almost finalized.
Scott Lab- Added bulk cap. added GND plane. Added lots of information on
the silkscreen. Barrel connectors for all power sources. Verified and
fixed programming header(added cap). Added barrel connectors to battery
PCB and made standoff drill holes.
Parts:
- removed X1: 22-23-2051, con-molex:22-23-2051
- added C1: 100uF, rcl:CPOL-USE3.5-8
- added I2C: 22-23-2021, con-molex:22-23-2021
- added U$7: 0.1uF, MinotaurParts:C-US-1206
- U$21: value 1k -> 470
- U$22: value 5k -> 10k
Connections:
- removed net N$60: SW_1.2, U$21.1
- new net N$79: SV5.7, U$1.*MCLR, U$21.2
- net +3V3: no longer X1-1.S
- net GND: now also C1.-, U$7.2; no longer X1-2.S
- net N$30: now also SW_1.2, U$21.1, U$7.1; no longer SV5.7, U$1.*MCLR, U$21.2
- net SCL: now also I2C-1.S; no longer X1-4.S
- net SDA: now also I2C-2.S; no longer X1-3.S
- net V+: now also C1.+
Other:
- note added: "SCL"
- note added: "SDA"
- moved on the sheet: U$21

Commit message: Finishing touches on PCB
Parts:
- X10: value MOTORS -> 22-23-2041
Changed lines of the file:
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@@
 <part name="SENSOR5" library="con-molex" deviceset="22-23-2031" device=""/>
 <part name="U$2" library="MinotaurParts" deviceset="L298" device=""/>
-<part name="X10" library="con-molex" deviceset="22-23-2041" device="" value="MOTORS"/>
+<part name="X10" library="con-molex" deviceset="22-23-2041" device="" value=""/>
 <part name="U$4" library="MinotaurParts" deviceset="TPS5450-Q1" device=""/>
 <part name="CBOOT7" library="MinotaurParts" deviceset="C-US-1206" device="" value="10nF"/>
